Commit message: ajout de urdf

File: 3rrr_robot_urdf/urdf/3rrr_robot_urdf.urdf (robot description, URDF)
Before this commit: robot 3rrr_robot_urdf, 8 links, 7 joints
Links:
- link base_link: geometry collision mesh filename=../meshes/base_link.STL; visual mesh filename=../meshes/base_link.STL
- link bras_avec_triange_3: geometry collision mesh filename=../meshes/bras_avec_triange_3.STL; visual mesh filename=../meshes/bras_avec_triange_3.STL
- link bras_avec_triangle_1: geometry collision mesh filename=../meshes/bras_avec_triangle_1.STL; visual mesh filename=../meshes/bras_avec_triangle_1.STL
- link bras_avec_triangle_2: geometry collision mesh filename=../meshes/bras_avec_triangle_2.STL; visual mesh filename=../meshes/bras_avec_triangle_2.STL
- link bras_ax12_1: geometry collision mesh filename=../meshes/bras_ax12_1.STL; visual mesh filename=../meshes/bras_ax12_1.STL
- link bras_ax12_2: geometry collision mesh filename=../meshes/bras_ax12_2.STL; visual mesh filename=../meshes/bras_ax12_2.STL
- link bras_ax12_3: geometry collision mesh filename=../meshes/bras_ax12_3.STL; visual mesh filename=../meshes/bras_ax12_3.STL
- link triangle: geometry collision mesh filename=../meshes/triangle.STL; visual mesh filename=../meshes/triangle.STL
